File: hardware/lorenz.kicad_sch (KiCad schematic)
At the start: 50 parts, among them J1 USB-C, J2 BNC, J3 BNC, J4 BNC, SW1 SW_DIP_x06, U1 LF412, U2 LF412, U3 MPY634, U4 MPY634, U5 A0515S-2WR2, U6 78L12, U7 79L12

Commit message: Schematic polish: project design rules, clean power section, owl plot
Design rules in the .kicad_pro are tighter than the cheapest tier at JLCPCB,
NextPCB and CircuitHub, so a board that passes DRC here passes at all three.
The owl's face on the sheet is the real trajectory, integrated by
lorenz_curve.py at s=10, r=28, b=8/3.

Co-Authored-By: Claude Opus 5 <noreply@anthropic.com>
Connections:
- net -12V: now also C15.1; no longer C15.2
- net -15V: now also C13.1; no longer C13.2
- net GND: now also C13.2, C15.2; no longer C13.1, C15.1
Other:
- moved on the sheet: C13, C15, D1, R13
