File: hardware/lorenz.kicad_sch (KiCad schematic)
At the start: 54 parts, among them J1 USB-C, J2 BNC, J3 BNC, J4 BNC, SW1 SW_DIP_x06, U1 LF412, U2 LF412, U3 MPY634, U4 MPY634, U5 A0515S-2WR2, U6 78L12, U7 79L12

Commit message: Use the isolation, add a chaos lamp and probe pads, drop the four-layer board
Circuit
 * The converter's isolation is now used.  GND (everything a scope touches)
   and GNDU (the USB input and its shell) are separate copper pours with a
   1 mm gap, bridged only by R21 = 1 M, C25 = 2.2 nF and JP1, an open solder
   jumper marked GND TIE.  The point is the ground loop: scope earth -> BNC
   shell -> board ground -> USB cable -> laptop -> earth, landing on signals
   whose full scale is 2 V.  U5 straddles the gap with its own barrier over it.
 * A common-cathode RGB lamp driven by x, -y and z, with its cathode held at
   -1.50 V by the half of U2 Paul never needed.  Holding the cathode below
   ground is what lets signals that swing either side of zero drive an LED:
   each colour lights above its own threshold, so red marks the +x wing, green
   the -x wing and blue brightens with z.  Resistors sized for equal perceived
   brightness, not equal current.
 * Three rail lamps -- yellow +5 V, green +12 V, white -12 V -- replacing one
   green LED that claimed "rails OK" while knowing nothing about two of them.
   All three are JLCPCB Basic parts, so the colours cost nothing.
 * Thirteen probe pads, each carrying on the silkscreen the name of what it
   probes, and three wire loops for a scope's ground clip.  Deliberately none
   on the summing junctions: they are virtual earths whose voltage is zero by
   construction, and a probe there is a 15 us pole on the integrator's input.

Board
 * The four-layer variant is gone.  Measured on the routed board: tracks cover
   1.2 % of the back copper, so the pour is already 98.8 % of an unbroken
   ground plane, against four times the bare-board price.
 * Two QR codes on the back, drawn by scripts/qrcode_gen.py, whose data
   placement and Reed-Solomon match the 'qrcode' package module for module and
   whose mask scoring matches segno's; check_outputs.py decodes them back out
   of the finished board on every build.
 * The switch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
Parts:
- added C24: 100nF, Capacitor_SMD:C_0805_2012Metric, symbol Device:C
- added C25: 2.2nF, Capacitor_SMD:C_0805_2012Metric, symbol Device:C
- added D2: green, LED_SMD:LED_0805_2012Metric, symbol Device:LED
- added D3: white, LED_SMD:LED_0805_2012Metric, symbol Device:LED
- added D4: RGB, lorenz:LED_RGB_PLCC4_3.5x2.8mm, symbol lorenz:LED_RGB_CC
- added JP1: GND TIE, Jumper:SolderJumper-2_P1.3mm_Open_Pad1.0x1.5mm, symbol Jumper:SolderJumper_2_Open
- added R14, R18, R19: 4.7k, Resistor_SMD:R_0805_2012Metric, symbol Device:R_US
- added R15: 10k, Resistor_SMD:R_0805_2012Metric, symbol Device:R_US
- added R16: 1.5k, Resistor_SMD:R_0805_2012Metric, symbol Device:R_US
- added R17: 6.8k, Resistor_SMD:R_0805_2012Metric, symbol Device:R_US
- added R20: 33k, Resistor_SMD:R_0805_2012Metric, symbol Device:R_US
- added R21: 1M, Resistor_SMD:R_0805_2012Metric, symbol Device:R_US
- added TP1: x, TestPoint:TestPoint_THTPad_D1.5mm_Drill0.7mm, symbol Connector:TestPoint
- added TP10: +12V, TestPoint:TestPoint_THTPad_D1.5mm_Drill0.7mm, symbol Connector:TestPoint
- added TP11: -12V, TestPoint:TestPoint_THTPad_D1.5mm_Drill0.7mm, symbol Connector:TestPoint
- added TP12: GND, TestPoint:TestPoint_THTPad_D1.5mm_Drill0.7mm, symbol Connector:TestPoint
- added TP13: GNDU, TestPoint:TestPoint_THTPad_D1.5mm_Drill0.7mm, symbol Connector:TestPoint
- added TP14, TP15, TP16: SCOPE GND, lorenz:ScopeGround_Loop, symbol Connector:TestPoint
- added TP2: -y, TestPoint:TestPoint_THTPad_D1.5mm_Drill0.7mm, symbol Connector:TestPoint
- added TP3: z, TestPoint:TestPoint_THTPad_D1.5mm_Drill0.7mm, symbol Connector:TestPoint
- added TP4: -xz/100, TestPoint:TestPoint_THTPad_D1.5mm_Drill0.7mm, symbol Connector:TestPoint
- added TP5: -xy/100, TestPoint:TestPoint_THTPad_D1.5mm_Drill0.7mm, symbol Connector:TestPoint
- added TP6: -1.5V, TestPoint:TestPoint_THTPad_D1.5mm_Drill0.7mm, symbol Connector:TestPoint
- added TP7: +5V, TestPoint:TestPoint_THTPad_D1.5mm_Drill0.7mm, symbol Connector:TestPoint
- added TP8: +15V, TestPoint:TestPoint_THTPad_D1.5mm_Drill0.7mm, symbol Connector:TestPoint
- added TP9: -15V, TestPoint:TestPoint_THTPad_D1.5mm_Drill0.7mm, symbol Connector:TestPoint
- D1: value green -> yellow; LCSC C2297 -> C2296; MPN KT-0805G -> KT-0805Y
- R13: value 4.7k -> 2.2k; LCSC C17673 -> C17520; MPN 0805W8F4701T5E -> 0805W8F2201T5E
Connections:
- net +12V: now also R14.1, TP10.1; no longer R13.1
- net +15V: now also TP8.1
- net +5V: now also R13.1, TP7.1
- net -12V: now also C15.2, R15.2, R20.2, TP11.1; no longer C15.1
- net -15V: now also C13.2, TP9.1; no longer C13.1
- net -y: now also R17.1, TP2.1
- net GND: now also C13.1, C15.1, C24.2, C25.2, D2.1 (K), D3.2 (A), JP1.2 (B), R19.2, R21.2, TP12.1, TP14.1, TP15.1, TP16.1; no longer C10.2, C11.2, C13.2, C15.2, D1.1 (K), J1.A1 (GND), J1.A12 (GND), J1.B1 (GND), J1.B12 (GND), J1.SH (SHIELD), R11.2, R12.2, U2.5 (+), U5.2 (-Vin)
- net x: now also R16.1, TP1.1
- net xy: now also TP5.1
- net xz: now also TP4.1
- net z: now also R18.1, TP3.1
- net SJ_X: now reaches C1.2, C2.2, C3.2, R1.2, R2.2, U1.2 (-)
- net SJ_Y: now reaches C4.2, C5.2, C6.2, R3.2, R4.2, R5.2, U1.6 (-)
- net SJ_Z: now reaches C7.2, C8.2, C9.2, R6.2, R7.2, U2.2 (-)
- net at U2.6 (-), U2.7: now also D4.4 (K), TP6.1
- new net: D3.1 (K), R15.1
- new net: D4.3 (G), R17.2
- new net: D4.1 (R), R16.2
- new net: D4.2 (B), R18.2
- new net: D2.2 (A), R14.2
- new net: C24.1, R19.1, R20.1, U2.5 (+)
- new net GNDU: C10.2, C11.2, C25.1, D1.1 (K), J1.A1 (GND), J1.A12 (GND), J1.B1 (GND), J1.B12 (GND), J1.SH (SHIELD), JP1.1 (A), R11.2, R12.2, R21.1, TP13.1, U5.2 (-Vin)
Other:
- note added: "-12 V x 4.7k / (4.7k + 33k) = -1.5 V, buffered so"
- note added: "-y -> green"
- note added: "1"
- note added: "102 ms"
- note added: "102 nF"
- note added: "2"
- note added: "2.2 ms"
- note added: "2.2 nF"
- note added: "3"
- note added: "4"
- note added: "472 ms"
- note added: "472 nF"
- note added: "5"
- note added: "6"
- note added: "CHAOS LAMP"
- note added: "GND"
- note added: "GNDU"
- note added: "ISOLATION BARRIER"
- note added: "JP1 open: the analog ground floats, and a scope's"
- note added: "Never both banks ON: that is 572 nF, which works but is not one of"
- note added: "ON"
- note added: "PROBE POINTS"
- note added: "RAIL LAMPS"
- note added: "SW1 pole"
- note added: "U2 z integrator + lamp buffer"
- note added: "a plated hole for a probe tip, one per rail, plus three wire"
- note added: "about 25 mA per rail; the 2 W module is rated +/-66 mA"
- note added: "common-mode current home. Bridge JP1 to give the"
- note added: "ground clip is what sets it -- so no mains-referenced"
- note added: "isolation up and tie the two grounds together."
- note added: "loop runs through the signal ground. 1 M drains"
- note added: "loops a scope's ground clip can bite on"
- note added: "off"
- note added: "on the USB side of the barrier"
- note added: "one per rail, three colours,"
- note added: "scope ground clips"
- note added: "shell and cable screen stay"
- note added: "so a dark one names itself"
- note added: "speed"
- note added: "static and 2.2 nF takes the converter's 100 kHz"
- note added: "tau = 1M x C"
- note added: "the lamp current cannot drag the reference about."
- note added: "the three settings the board is labelled for."
- note added: "x -> red"
- note added: "z -> blue"
- note removed: "LF412s too. An unused op-amp is parked as a"
- note removed: "SW1-1,2,3 ON SW1-4,5,6 off C = 102 nF nice! tau = 102 ms"
- note removed: "SW1-1,2,3 off SW1-4,5,6 ON C = 472 nF slow! tau = 472 ms"
- note removed: "SW1-1,2,3 off SW1-4,5,6 off C = 2.2 nF fast! tau = 2.2 ms"
- note removed: "U2 z integrator (B half spare)"
- note removed: "U2B is spare -- Paul only needed one and a half"
- note removed: "about 20 mA per rail; the 2 W module is rated +/-66 mA"
- note removed: "input ground -- the"
- note removed: "isolation is not used"
- note removed: "output common tied to"
- note removed: "rails OK"
- note removed: "shell grounded here only"
- note removed: "unity-gain follower with its input grounded."
- moved on the sheet: C13, C15, D1, R13, U2B

Commit message: Rebuild the board around the multipliers, and review the whole design
Layout.  The multipliers move to the far left, into the third of the board
that was empty, and everything spreads out behind them.  Each output row is
now one straight line -- op-amp, probe pad, the 100 ohm lying horizontally,
BNC -- so what the probe pad is for needs no explaining.  The switch legend
gets clear board around it, both multipliers and both op-amps say what they
are, the chaos lamp has its own quarter with its resistors coming in from the
left, and the two QR codes are 62 mm apart with no drilled hole in either.

The lamp is redrawn: each colour is fed from its own integrator's *output*
node, tapped between the op-amp and the 100 ohm series resistor and brought
down the right margin, so there is no way to read it as current taken from an
op-amp input.  The three rail lamps are gone -- the chaos lamp cannot light
unless every rail is up, so it is the power-on indicator.

Review.  Four bugs, worst first.  DRC had never read this project's design
rules: pcbnew writes a default .kicad_pro beside any board it saves and
make.py only put the real one back after DRC ran, so every "0 violations" was
measured against KiCad's defaults.  The real rules turned up 203 violations.
Then: every via was 0.15 mm of annulus against a 0.25 mm rule; stitching vias
were leaving 0.08 mm necks of copper beside through-hole pads, which are
their own vias anyway; and the legend placer avoided pads but not package
bodies, so both multipliers had their designators printed underneath them.

New checks that run every build: check_pinout.py writes each IC's pin table
from its datasheet, compares it with the symbol used here, and compares it
again with KiCad's own library where the same part exists; gen_pcb.py refuses
to build if any net has pads on both sides of the isolation gap or any track
crosses it.  Four 100 nF parts now sit at the regulators' own pins, which is
what those datasheets are characterised with.

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
Parts:
- removed D2: green, LED_SMD:LED_0805_2012Metric, symbol Device:LED
- removed D3: white, LED_SMD:LED_0805_2012Metric, symbol Device:LED
- removed D4: RGB, lorenz:LED_RGB_PLCC4_3.5x2.8mm, symbol lorenz:LED_RGB_CC
- removed R19: 4.7k, Resistor_SMD:R_0805_2012Metric, symbol Device:R_US
- removed R20: 33k, Resistor_SMD:R_0805_2012Metric, symbol Device:R_US
- removed R21: 1M, Resistor_SMD:R_0805_2012Metric, symbol Device:R_US
- added C26, C27, C28, C29: 100nF, Capacitor_SMD:C_0805_2012Metric, symbol Device:C
- D1: value yellow -> RGB; footprint LED_SMD:LED_0805_2012Metric -> lorenz:LED_RGB_PLCC4_3.5x2.8mm; symbol Device:LED -> lorenz:LED_RGB_CC; LCSC C2296 -> C2962096; MPN KT-0805Y -> MHPC3528CRGBCT
- F1: footprint Fuse:Fuse_1812_4532Metric -> lorenz:PTC_1812_4532Metric
- R13: value 2.2k -> 1.5k; LCSC C17520 -> C4310; MPN 0805W8F2201T5E -> 0805W8F1501T5E
- R14: value 4.7k -> 6.8k; LCSC C17673 -> C17772; MPN 0805W8F4701T5E -> 0805W8F6801T5E
- R15: value 10k -> 4.7k; LCSC C17414 -> C17673; MPN 0805W8F1002T5E -> 0805W8F4701T5E
- R16: value 1.5k -> 4.7k; LCSC C4310 -> C17673; MPN 0805W8F1501T5E -> 0805W8F4701T5E
- R17: value 6.8k -> 33k; LCSC C17772 -> C17633; MPN 0805W8F6801T5E -> 0805W8F3302T5E
- R18: value 4.7k -> 1M; LCSC C17673 -> C17514; MPN 0805W8F4701T5E -> 0805W8F1004T5E
- TP14, TP15, TP16: footprint lorenz:ScopeGround_Loop -> lorenz:TestPoint_ScopeGnd_Loop_2x1.1mm
Connections:
- net +12V: now also C27.2; no longer R14.1
- net +15V: now also C26.2
- net +5V: no longer R13.1
- net -12V: now also R17.1, C29.1; no longer R15.2
- net -15V: now also C28.1
- net -y: now also R14.2; no longer R17.1
- net GND: now also R16.2, R18.2, C26.1, C27.1, C28.2, C29.2
- net GNDU: now also R18.1; no longer D1.1 (K)
- net x: now also R13.2; no longer R16.1
- net z: now also R15.2; no longer R18.1
- net at R15.1: now also D1.2 (B)
- net at TP6.1, U2.6 (-), U2.7: now also D1.4 (K)
- net at R17.2: now also C24.1, R16.1, U2.5 (+)
- new net: D1.1 (R), R13.1
- new net: D1.3 (G), R14.1
Other:
- note added: "-12 V x 4.7k / (4.7k + 33k) = -1.5 V, buffered by U2B -- the half"
- note added: "100 kHz common-mode current home."
- note added: "Bridge JP1 to give the isolation up."
- note added: "JP1 open: the analog ground floats,"
- note added: "One lamp, three colours, driven from the three outputs."
- note added: "and a scope's ground clip is what sets"
- note added: "cathode. Putting the cathode below ground is what lets a signal"
- note added: "it, so no mains-referenced loop runs"
- note added: "of the LF412 Paul never needed -- and held on the lamp's common"
- note added: "one lights only above its own turn-on voltage. The taps are on"
- note added: "resistor, so no lamp current flows in the BNC output impedance."
- note added: "static; 2.2 nF takes the converter's"
- note added: "that swings either side of zero switch a colour on and off: each"
- note added: "the output side of each integrator, ahead of the 100 ohm series"
- note added: "through the signal ground. 1 M drains"
- note removed: "-12 V x 4.7k / (4.7k + 33k) = -1.5 V, buffered so"
- note removed: "JP1 open: the analog ground floats, and a scope's"
- note removed: "RAIL LAMPS"
- note removed: "common-mode current home. Bridge JP1 to give the"
- note removed: "ground clip is what sets it -- so no mains-referenced"
- note removed: "isolation up and tie the two grounds together."
- note removed: "loop runs through the signal ground. 1 M drains"
- note removed: "one per rail, three colours,"
- note removed: "so a dark one names itself"
- note removed: "static and 2.2 nF takes the converter's 100 kHz"
- note removed: "the lamp current cannot drag the reference about."
- moved on the sheet: C24, R13, R14, R15, R16, R17, R18, U2B

Commit message: Add an r knob and a sync input, and build the lamp as option 038
The lamp is now the common-anode MHPA3528CRGBCT held at +3.20 V by U2B,
with z -> red through 470R, x -> green through 3.9k and -y -> blue
through 1.5k: option 038 of the hundred renderings.  All three peaks land
within 8 % of each other, so the colour mixes instead of blinking.

R3 splits into 27k plus RV1, a Bourns 3386P 20k trimmer, sweeping
r = 21.3 to 37.0 across both bifurcations and Lorenz's 28.  Terminal 1 is
tied to the wiper, so grit under the wiper means maximum resistance and
the lowest r, never an open circuit.  check_circuit.py now solves the
whole board twice, once at each end of the knob, and checks r as a range.

A SYNC IN pad feeds the dy/dt summing junction through 100k, with 1M
holding it down when nothing is plugged in.  That junction is the only
one where an inverting input can still add to a term: drive it from
another board's x, turn the receiver's knob down by 10, and the two lock
in about five time units.  Pull the wire and they diverge again, which is
what the freeze switch was going to be for.

Also: a filled pin-1 triangle on every part that can be fitted turned,
drawn from the real pad and courtyard; every series resistor rotated
horizontal to match the schematic and every shunt vertical; the USB-C
moved 4 mm out so a cable with a moulded body can seat; a fourth speed
called "glacial!"; the x/y/z -> R/G/B mapping on the front silk beside
the lamp; URLs printed under both QR codes; and the back paragraph reset
one sentence per line across the foot of the board.

Co-Authored-By: Claude Opus 5 <noreply@anthropic.com>
Parts:
- added R19: 100k, Resistor_SMD:R_0805_2012Metric, symbol Device:R_US
- added R20: 1M, Resistor_SMD:R_0805_2012Metric, symbol Device:R_US
- added RV1: 20k, lorenz:Potentiometer_Bourns_3386P_Vertical, symbol Device:R_Potentiometer_Trim_US
- added TP17: SCOPE GND, lorenz:TestPoint_ScopeGnd_Loop_2x1.1mm, symbol Connector:TestPoint
- D1: symbol lorenz:LED_RGB_CC -> lorenz:LED_RGB_CA; LCSC C2962096 -> C2962095; MPN MHPC3528CRGBCT -> MHPA3528CRGBCT
- R13: value 1.5k -> 3.9k; LCSC C4310 -> C17614; MPN 0805W8F1501T5E -> 0805W8F3901T5E
- R14: value 6.8k -> 1.5k; LCSC C17772 -> C4310; MPN 0805W8F6801T5E -> 0805W8F1501T5E
- R15: value 4.7k -> 470R; LCSC C17673 -> C17710; MPN 0805W8F4701T5E -> 0805W8F4700T5E
- R16: value 4.7k -> 12k; LCSC C17673 -> C17444; MPN 0805W8F4701T5E -> 0805W8F1202T5E
- R3: value 35.7k -> 27k; LCSC C843989 -> C17593; MPN CRCW080535K7FKEA -> 0805W8F2702T5E
- TP10: value +12V -> -15V
- TP11: value -12V -> +12V
- TP12: value GND -> -12V
- TP13: value GNDU -> GND
- TP14: value SCOPE GND -> GNDU; footprint lorenz:TestPoint_ScopeGnd_Loop_2x1.1mm -> TestPoint:TestPoint_THTPad_D1.5mm_Drill0.7mm
- TP4: value -xz/100 -> SYNC IN
- TP5: value -xy/100 -> -xz/100
- TP6: value -1.5V -> -xy/100
- TP7: value +5V -> +3.2V
- TP8: value +15V -> +5V
- TP9: value -15V -> +15V
Connections:
- net +12V: now also R17.1, TP11.1; no longer TP10.1
- net +15V: now also TP9.1; no longer TP8.1
- net +5V: now also TP8.1; no longer TP7.1
- net -12V: now also TP12.1; no longer R17.1, TP11.1
- net -15V: now also TP10.1; no longer TP9.1
- net GND: now also TP13.1, R20.2, TP17.1; no longer TP12.1, TP14.1
- net GNDU: now also TP14.1; no longer TP13.1
- net SJ_Y: now also R19.2
- net x: now also RV1.1, RV1.2; no longer R3.1
- net xy: now also TP6.1; no longer TP5.1
- net xz: now also TP5.1; no longer TP4.1
- net at R15.1: now also D1.4 (R); no longer D1.2 (B)
- net at D1.1 (A): now also TP7.1, U2.6 (-), U2.7; no longer R13.1
- net at R14.1: now also D1.2 (B); no longer D1.3 (G)
- new net: D1.3 (G), R13.1
- new net: R3.1, RV1.3
- new net: R19.1, R20.1, TP4.1
Other:
- note added: "+12 V x 12k / (12k + 33k) = +3.2 V, buffered by U2B -- the half"
- note added: "-y -> blue"
- note added: "100 % r = 37 wings still there, orbit tighter and faster"
- note added: "1M holds the pad at 0 V"
- note added: "27 % r = 24.06 below this, the trace spirals into one wing"
- note added: "33 % r = 24.74 above this, both fixed points are unstable"
- note added: "56 % r = 28 Lorenz's own value -- the owl's face"
- note added: "572 ms"
- note added: "572 nF"
- note added: "All four are printed on the back of the board, next to the switch."
- note added: "Between 27 % and 33 % -- eighteen degrees of screw -- chaos and"
- note added: "Clockwise raises r, and 310 degrees of screw covers 21.3 to 37.0:"
- note added: "ON adds a fourth speed Paul never had, slow enough to watch by eye."
- note added: "R19 = 100k sets the coupling to 1M/100k = 10. It lands on the r x"
- note added: "R3 + RV1 = 27k + (20k..0) -> 1M/47k .. 1M/27k = 21.3 .. 37.0 = r"
- note added: "RV1 is the only control that changes the shape of the attractor."
- note added: "Run a wire from one board's x output to a second board's SYNC IN pad."
- note added: "SYNCHRONISING TWO BOARDS"
- note added: "THE r KNOB"
- note added: "The knob is wired as a rheostat, terminal 3 and the wiper, with"
- note added: "Within a few seconds the second board is drawing the first board's"
- note added: "anode. Each die then lights when its own signal goes low, and"
- note added: "colour wanders through mixed hues rather than blinking between"
- note added: "current flows in the BNC output impedance."
- note added: "degree, so a few percent of knob is a visible change and you can"
- note added: "depends on where you started. Elsewhere r moves about 0.05 per"
- note added: "dy/dt = r x - y - x z"
- note added: "equations. That offset is why the knob spans more than 10."
- note added: "fail open, and this one is not trusted not to."
- note added: "for s to absorb it with. z never locks at any strength -- the x, y"
- note added: "glacial!"
- note added: "goes to its minimum instead of the r x term disappearing. Wipers"
- note added: "integrator, ahead of the 100 ohm series resistor, so no lamp"
- note added: "lifts the wiper, the whole 20k track still bridges the branch, so r"
- note added: "offset. -y would lock too, into the top of R1, but there is no knob"
- note added: "one case Pecora and Carroll's 1990 paper says must fail. Try it."
- note added: "pair driven by z keeps a positive conditional Lyapunov exponent, the"
- note added: "r knob"
- note added: "saturated primaries. The taps are on the output side of each"
- note added: "still find your way back to a setting you liked."
- note added: "stocks a 3-pole 3-position switch; 2.2 nF is always fitted. Both banks"
- note added: "term, so it also adds 10 to the receiving board's r: set the driver"
- note added: "terminal 1 tied to the wiper. That short is the point: if grit ever"
- note added: "that agree to a few millivolts, and completely different futures"
- note added: "the three come within 5 % of the same peak brightness, so the"
- note added: "the two fixed points are both stable, and which one you land in"
- note added: "to r = 32 and the receiver to r = 22 and both are solving the same"
- note added: "trajectory, whatever state it was in when you connected it. Pull the"
- note added: "when nothing is plugged in"
- note added: "wire off and the two drift apart again: the same equations, states"
- note added: "within a minute. That is the demonstration, and it needs no switch."
- note added: "x -> green"
- note added: "x is the channel that gets a pad because the knob can absorb the"
- note added: "z -> red"
- note removed: "-12 V x 4.7k / (4.7k + 33k) = -1.5 V, buffered by U2B -- the half"
- note removed: "-y -> green"
- note removed: "Never both banks ON: that is 572 nF, which works but is not one of"
- note removed: "R3 = 35.7k -> 1M/35.7k = 28.01 = r"
- note removed: "cathode. Putting the cathode below ground is what lets a signal"
- note removed: "dy/dt = 28 x - y - x z"
- note removed: "one lights only above its own turn-on voltage. The taps are on"
- note removed: "resistor, so no lamp current flows in the BNC output impedance."
- note removed: "stocks a 3-pole 3-position switch; 2.2 nF is always fitted."
- note removed: "that swings either side of zero switch a colour on and off: each"
- note removed: "the output side of each integrator, ahead of the 100 ohm series"
- note removed: "the three settings the board is labelled for."
- note removed: "x -> red"
- note removed: "z -> blue"
