File: hardware/lorenz.kicad_sch (KiCad schematic)
At the start: 86 parts, among them J1 USB-C, J2 BNC, J3 BNC, J4 BNC, SW1 SW_DIP_x06, U1 LF412, U2 LF412, U3 MPY634, U4 MPY634, U5 A0515S-2WR2, U6 78L12, U7 79L12

Commit message: Say what the sync input needs, and give the notes room to say it
Two boards both float on purpose, so a bare wire from one board's x to
the other's SYNC IN does nothing without a ground in common.  The
schematic, DESIGN_NOTES and the response all say so now, and say that a
coax screen from a BNC splitter does both jobs at once.

Also corrects the reason z cannot be a sync channel.  It is not a
conditional-Lyapunov obstruction -- sign-correct diffusive coupling on z
does lock in simulation -- it is that the summing junction inverts, so an
injected z arrives with a minus sign and drives the two boards apart.
Getting the plus sign would need a -z output this circuit does not make.

The lamp notes were claiming peaks within 5 %; the model says 8 %, with
green and blue lit 87 % and 84 % of the time and red 28 %.  Fixed
everywhere, along with the title block's "r = 28", which is now a range.

Co-Authored-By: Claude Opus 5 <noreply@anthropic.com>
Other:
- note added: "R19 = 100k makes the coupling 1M/100k = 10. It lands on the r x"
- note added: "Run a wire from one board's x output to a second board's SYNC IN"
- note added: "That offset is why the knob spans more than 10."
- note added: "arrives with a minus sign and drives the two boards apart. The plus"
- note added: "both at once. Both boards float, so with no common ground nothing"
- note added: "few millivolts. That is the demonstration, and it needs no switch."
- note added: "happens at all."
- note added: "pad, and tie the two analog grounds together -- a coax screen does"
- note added: "r = 32, receive at r = 22, and both are solving the same equations."
- note added: "sign would need a -z output, and this circuit does not make one."
- note added: "term, so it also adds 10 to the receiving board's r: drive at"
- note added: "the three peaks land within 8 % of each other, so the colour"
- note added: "too, but only with R1 changed as well, and there is no knob for s."
- note added: "wanders through mixed hues rather than blinking between"
- note added: "wire off and the two drift apart again from states that agree to a"
- note added: "with nothing plugged in"
- note added: "x gets the pad because the knob absorbs that offset. -y would lock"
- note added: "z cannot be done at all: the junction inverts, so an injected z"
- note removed: "R19 = 100k sets the coupling to 1M/100k = 10. It lands on the r x"
- note removed: "Run a wire from one board's x output to a second board's SYNC IN pad."
- note removed: "colour wanders through mixed hues rather than blinking between"
- note removed: "equations. That offset is why the knob spans more than 10."
- note removed: "for s to absorb it with. z never locks at any strength -- the x, y"
- note removed: "offset. -y would lock too, into the top of R1, but there is no knob"
- note removed: "one case Pecora and Carroll's 1990 paper says must fail. Try it."
- note removed: "pair driven by z keeps a positive conditional Lyapunov exponent, the"
- note removed: "term, so it also adds 10 to the receiving board's r: set the driver"
- note removed: "that agree to a few millivolts, and completely different futures"
- note removed: "the three come within 5 % of the same peak brightness, so the"
- note removed: "to r = 32 and the receiver to r = 22 and both are solving the same"
- note removed: "when nothing is plugged in"
- note removed: "wire off and the two drift apart again: the same equations, states"
- note removed: "within a minute. That is the demonstration, and it needs no switch."
- note removed: "x is the channel that gets a pad because the knob can absorb the"
- moved on the sheet: R19, R20

Commit message: Give SYNC IN X its own BNC, a weight knob, and a drawing that adds up
SYNC IN is now SYNC IN X everywhere: a fourth BNC on the left edge, in
line with the x output on the right, because another board's x output is
what goes in it.  RV2 sets how much of it gets in.

RV2 is a divider across the incoming signal rather than a rheostat in
series with R19, which makes the weight linear in the knob --
g = 1M/100k x (fraction turned) = 0 to 10 -- instead of hyperbolic.  A
rheostat would have crammed the locking threshold, about g = 7, into the
first tenth of the rotation; as a divider it lands at 70 %, so the bottom
seven tenths is "never quite" and the top three tenths locks in a couple
of seconds at slow!.  At the counter-clockwise stop the wiper sits on
ground and the branch contributes nothing, which is the same thing as
unplugging the cable.

The drawing now says what the circuit means.  Row 2's branches run -y,
x z, x down the sheet, and the x branch and the sync branch join on their
own rail before that rail reaches the summing junction: a perturbation on
the x term, not a fourth term.  On the board R19 is the next resistor
down the column from R3, with "SYNC IN X adds here" beside it, and the
whole chain -- jack, knob, resistor -- runs left to right into the
column.  The multipliers moved 9 mm right to make room, and the back's
equations shrank to clear the drilled parts down that edge.

Also: the pin-1 triangles are back to the four parts whose own footprints
have no legible mark (D1, SW1, RV1, RV2) rather than every rotatable
part; poles 1-3 now carry the 470 nF and 4-6 the 100 nF so the six
sliders read left to right as a binary number; "glacial!" is "slower!";
the credit line and the circuit URL swapped places, with the date and
revision under the credit at 0.9 mm; and the owl caption says 'scope.

Co-Authored-By: Claude Opus 5 <noreply@anthropic.com>
Parts:
- removed TP17: SCOPE GND, lorenz:TestPoint_ScopeGnd_Loop_2x1.1mm, symbol Connector:TestPoint
- added J5: BNC, lorenz:BNC_KYWE_RightAngle, symbol Connector:Conn_Coaxial
- added RV2: 20k, lorenz:Potentiometer_Bourns_3386P_Vertical, symbol Device:R_Potentiometer_Trim_US
- TP10: value -15V -> +12V
- TP11: value +12V -> -12V
- TP12: value -12V -> GND
- TP13: value GND -> GNDU
- TP14: value GNDU -> SCOPE GND; footprint TestPoint:TestPoint_THTPad_D1.5mm_Drill0.7mm -> lorenz:TestPoint_ScopeGnd_Loop_2x1.1mm
- TP4: value SYNC IN -> -xz/100
- TP5: value -xz/100 -> -xy/100
- TP6: value -xy/100 -> +3.2V
- TP7: value +3.2V -> +5V
- TP8: value +5V -> +15V
- TP9: value +15V -> -15V
Connections:
- net +12V: now also TP10.1; no longer TP11.1
- net +15V: now also TP8.1; no longer TP9.1
- net +5V: now also TP7.1; no longer TP8.1
- net -12V: now also TP11.1; no longer TP12.1
- net -15V: now also TP9.1; no longer TP10.1
- net GND: now also R20.1, TP12.1, TP14.1, J5.2 (Ext), RV2.1; no longer R20.2, TP13.1
- net GNDU: now also TP13.1; no longer TP14.1
- net xy: now also TP5.1; no longer TP6.1
- net xz: now also TP4.1; no longer TP5.1
- net at D1.1 (A), U2.6 (-), U2.7: now also TP6.1; no longer TP7.1
- net at C8.1: now also SW1.6; no longer SW1.3
- net at C2.1: now also SW1.4; no longer SW1.1
- net at C9.1: now also SW1.3; no longer SW1.6
- net at C5.1: now also SW1.5; no longer SW1.2
- net at C3.1: now also SW1.1; no longer SW1.4
- net at C6.1: now also SW1.2; no longer SW1.5
- new net: J5.1 (In), RV2.3
- new net: R19.1, R20.2, RV2.2
Other:
- note added: "0 .. 10"
- note added: "1M holds this node at 0 V if the wiper lifts"
- note added: "470 nF and poles 4-6 the 100 nF, so the six sliders read left to"
- note added: "ON adds a fourth speed Paul never had. Poles 1-3 switch in the"
- note added: "RV2 is a divider across the incoming signal, so the weight is linear"
- note added: "Run a cable from one board's x output to a second board's SYNC IN X"
- note added: "SYNC IN X"
- note added: "The coupling lands on the r x term, so it also adds g to the"
- note added: "The knob is a rheostat, terminal 3 and the wiper, with terminal 1"
- note added: "Turn the weight knob up and within a few seconds the second board is"
- note added: "arrives with a minus sign and drives the boards apart; the plus sign"
- note added: "couple of seconds. At the counter-clockwise stop the wiper is on"
- note added: "degree, so you can find a setting you liked again."
- note added: "demonstration, and it needs no switch."
- note added: "drawing the first board's trajectory, whatever state it was in when"
- note added: "from another board's x"
- note added: "from states that agree to a few millivolts. That is the whole"
- note added: "g = 7 they never lock however long you wait; above it they lock in a"
- note added: "ground and the branch contributes nothing, exactly as if unplugged."
- note added: "in the knob: g = 1M/100k x (fraction turned) = 0 to 10. Below about"
- note added: "its minimum instead of the r x term disappearing."
- note added: "jack, and tie the two analog grounds together -- a coax screen does"
- note added: "reads 32 down to 22 as the sync knob goes 0 to full."
- note added: "receiving board's own r: drive at r = 32 and the receiver's r knob"
- note added: "right as a two-digit binary number counting 00, 01, 10, 11."
- note added: "slower!"
- note added: "tied to the wiper. That short is the point: if grit ever lifts the"
- note added: "weight"
- note added: "wiper, the whole 20k track still bridges the branch, so r goes to"
- note added: "would need a -z output, and this circuit does not make one."
- note added: "x gets the jack because the knob absorbs that offset. -y would lock"
- note added: "you connected it. Pull the cable off and the two drift apart again"
- note removed: "1M holds the pad at 0 V"
- note removed: "ON adds a fourth speed Paul never had, slow enough to watch by eye."
- note removed: "R19 = 100k makes the coupling 1M/100k = 10. It lands on the r x"
- note removed: "Run a wire from one board's x output to a second board's SYNC IN"
- note removed: "That offset is why the knob spans more than 10."
- note removed: "The knob is wired as a rheostat, terminal 3 and the wiper, with"
- note removed: "Within a few seconds the second board is drawing the first board's"
- note removed: "arrives with a minus sign and drives the two boards apart. The plus"
- note removed: "degree, so a few percent of knob is a visible change and you can"
- note removed: "fail open, and this one is not trusted not to."
- note removed: "few millivolts. That is the demonstration, and it needs no switch."
- note removed: "glacial!"
- note removed: "goes to its minimum instead of the r x term disappearing. Wipers"
- note removed: "lifts the wiper, the whole 20k track still bridges the branch, so r"
- note removed: "pad, and tie the two analog grounds together -- a coax screen does"
- note removed: "r = 32, receive at r = 22, and both are solving the same equations."
- note removed: "sign would need a -z output, and this circuit does not make one."
- note removed: "still find your way back to a setting you liked."
- note removed: "term, so it also adds 10 to the receiving board's r: drive at"
- note removed: "terminal 1 tied to the wiper. That short is the point: if grit ever"
- note removed: "trajectory, whatever state it was in when you connected it. Pull the"
- note removed: "wire off and the two drift apart again from states that agree to a"
- note removed: "with nothing plugged in"
- note removed: "x gets the pad because the knob absorbs that offset. -y would lock"
- moved on the sheet: R19, R20, R5, SW1A, SW1B, SW1C, SW1D, SW1E, SW1F

Commit message: Four BNCs now, not three, in the mounting note
Co-Authored-By: Claude Opus 5 <noreply@anthropic.com>
Other:
- note added: "but with four BNCs around the edges the cables lever on the"
- note removed: "but with three BNCs along one edge the cables lever on the"

Commit message: Put the USB-C where its drawing says, not where DRC preferred
The HRO recommended layout puts the board edge 5.79 mm in front of the
upper shell-tab centre, so the connector's mating face overhangs the edge
by 0.99 mm.  Two other numbers in the same chain -- 1.64 from the signal
pad row to the upper tab, 4.18 between the tabs -- match KiCad's land
pattern exactly, so the datum is certain.

The board had the edge at +4.15 instead of +2.66: the face sat half a
millimetre inside the laminate, which is the thing a moulded plug body
hits.  The reason is the mistake worth recording.  In prompt 4 the
footprint's silkscreen ran past where the edge had to be, DRC objected,
and the connector was moved until DRC went quiet -- letting a drawing
rule overrule a mechanical dimension.

lorenz.pretty now carries its own copy of the footprint: KiCad's land
pattern untouched, the two silkscreen segments that would print off the
board trimmed at +2.45, and the local 3D model baked in instead of
swapped on at board level.  J1 moves to y = 97.34, DRC stays at zero, and
copper comes no closer than 0.81 mm to the edge.

check_outputs re-derives the requirement from the placed shell tabs on
every build, so the dimension cannot drift a third time.

Co-Authored-By: Claude Opus 5 <noreply@anthropic.com>
Parts:
- J1: footprint Connector_USB:USB_C_Receptacle_HRO_TYPE-C-31-M-12 -> lorenz:USB_C_Receptacle_HRO_TYPE-C-31-M-12
Changed lines of the file:
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@@
 			)
 		)
-		(property "Footprint" "Connector_USB:USB_C_Receptacle_HRO_TYPE-C-31-M-12"
+		(property "Footprint" "lorenz:USB_C_Receptacle_HRO_TYPE-C-31-M-12"
 			(at 45.72 340.36 0)
 			(hide yes)
