File: hardware/lorenz-4layer.kicad_pcb (KiCad board)
At the start: 4 copper layers, 100 x 100 mm, 50 parts, among them J1 USB-C, J2 BNC, J3 BNC, J4 BNC, SW1 SW_DIP_x06, U1 LF412, U2 LF412, U3 MPY634, U4 MPY634, U5 A0515S-2WR2, U6 78L12, U7 79L12

Commit message: M3 mounting holes, and a schematic layout checker that caught their caption
check_schematic.py estimates every text item's extent from KiCad's stroke font
and reports overlaps, strays outside the frame, and anything landing in the
title block.  It found the one note that had drifted off the left edge, and
then immediately caught the mounting-hole caption when I dropped it on top of
the title block.

Co-Authored-By: Claude Opus 5 <noreply@anthropic.com>
Parts:
- added MH1: MountingHole, MountingHole:MountingHole_3.2mm_M3, F.Cu at (4.00, 4.00)
- added MH2: MountingHole, MountingHole:MountingHole_3.2mm_M3, F.Cu at (96.0, 4.00)
- added MH3: MountingHole, MountingHole:MountingHole_3.2mm_M3, F.Cu at (4.00, 96.0)
- added MH4: MountingHole, MountingHole:MountingHole_3.2mm_M3, F.Cu at (96.0, 96.0)
- moved D1 6.00 mm to (88.0, 96.0)
- moved R13 2.00 mm to (82.0, 96.0)
Routing:
- net Net-(D1-A): track 10.0 -> 6.01 mm
- net +12V: track 172.5 -> 172.1 mm, vias 13 -> 14
- net GND: vias 378 -> 375
