File: hardware/lorenz-4layer.kicad_sch (KiCad schematic)
At the start: 50 parts, among them J1 USB-C, J2 BNC, J3 BNC, J4 BNC, SW1 SW_DIP_x06, U1 LF412, U2 LF412, U3 MPY634, U4 MPY634, U5 A0515S-2WR2, U6 78L12, U7 79L12

Commit message: M3 mounting holes, and a schematic layout checker that caught their caption
check_schematic.py estimates every text item's extent from KiCad's stroke font
and reports overlaps, strays outside the frame, and anything landing in the
title block.  It found the one note that had drifted off the left edge, and
then immediately caught the mounting-hole caption when I dropped it on top of
the title block.

Co-Authored-By: Claude Opus 5 <noreply@anthropic.com>
Parts:
- added MH1, MH2, MH3, MH4: MountingHole, MountingHole:MountingHole_3.2mm_M3, symbol Mechanical:MountingHole
Other:
- note added: "Four M3 holes, one per board corner. No electrical function,"
- note added: "MOUNTING"
- note added: "board, so it wants standoffs rather than a bare bench."
- note added: "but with three BNCs along one edge the cables lever on the"
