File: hardware/lorenz-4layer.kicad_sch (KiCad schematic)
At the start: 54 parts, among them J1 USB-C, J2 BNC, J3 BNC, J4 BNC, SW1 SW_DIP_x06, U1 LF412, U2 LF412, U3 MPY634, U4 MPY634, U5 A0515S-2WR2, U6 78L12, U7 79L12

Commit message: Count solder joints, not mounting holes; quote the time constants directly
Co-Authored-By: Claude Opus 5 <noreply@anthropic.com>
Other:
- note added: "SW1-1,2,3 ON SW1-4,5,6 off C = 102 nF nice! tau = 102 ms"
- note added: "SW1-1,2,3 off SW1-4,5,6 ON C = 472 nF slow! tau = 472 ms"
- note added: "SW1-1,2,3 off SW1-4,5,6 off C = 2.2 nF fast! tau = 2.2 ms"
- note removed: "SW1-1,2,3 ON SW1-4,5,6 off C = 102 nF nice! ~0.15 s per lobe"
- note removed: "SW1-1,2,3 off SW1-4,5,6 ON C = 472 nF slow! ~0.7 s per lobe"
- note removed: "SW1-1,2,3 off SW1-4,5,6 off C = 2.2 nF fast! ~3 ms per lobe"
Changed lines of the file:
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@@
 		)
 	)
-	(text "SW1-1,2,3 ON    SW1-4,5,6 off   C = 102 nF     nice!   ~0.15 s per lobe"
+	(text "SW1-1,2,3 ON    SW1-4,5,6 off   C = 102 nF     nice!   tau = 102 ms"
 		(exclude_from_sim no)
 		(at 293 296 0)
@@
 		)
 	)
-	(text "SW1-1,2,3 off   SW1-4,5,6 ON    C = 472 nF     slow!   ~0.7 s per lobe"
+	(text "SW1-1,2,3 off   SW1-4,5,6 ON    C = 472 nF     slow!   tau = 472 ms"
 		(exclude_from_sim no)
 		(at 293 300.2 0)
@@
 		)
 	)
-	(text "SW1-1,2,3 off   SW1-4,5,6 off   C = 2.2 nF     fast!   ~3 ms per lobe"
+	(text "SW1-1,2,3 off   SW1-4,5,6 off   C = 2.2 nF     fast!   tau = 2.2 ms"
 		(exclude_from_sim no)
 		(at 293 291.8 0)
