File: hardware/lorenz.kicad_pcb (KiCad board)
At the start: 2 copper layers, 100 x 100 mm, 87 parts, among them J1 USB-C, J2 BNC, J3 BNC, J4 BNC, J5 BNC, SW1 SW_DIP_x06, U1 LF412, U2 LF412, U3 MPY634, U4 MPY634, U5 A0515S-2WR2, U6 78L12, U7 79L12

Commit message: Put the USB-C where its drawing says, not where DRC preferred
The HRO recommended layout puts the board edge 5.79 mm in front of the
upper shell-tab centre, so the connector's mating face overhangs the edge
by 0.99 mm.  Two other numbers in the same chain -- 1.64 from the signal
pad row to the upper tab, 4.18 between the tabs -- match KiCad's land
pattern exactly, so the datum is certain.

The board had the edge at +4.15 instead of +2.66: the face sat half a
millimetre inside the laminate, which is the thing a moulded plug body
hits.  The reason is the mistake worth recording.  In prompt 4 the
footprint's silkscreen ran past where the edge had to be, DRC objected,
and the connector was moved until DRC went quiet -- letting a drawing
rule overrule a mechanical dimension.

lorenz.pretty now carries its own copy of the footprint: KiCad's land
pattern untouched, the two silkscreen segments that would print off the
board trimmed at +2.45, and the local 3D model baked in instead of
swapped on at board level.  J1 moves to y = 97.34, DRC stays at zero, and
copper comes no closer than 0.81 mm to the edge.

check_outputs re-derives the requirement from the placed shell tabs on
every build, so the dimension cannot drift a third time.

Co-Authored-By: Claude Opus 5 <noreply@anthropic.com>
Parts:
- J1: footprint Connector_USB:USB_C_Receptacle_HRO_TYPE-C-31-M-12 -> lorenz:USB_C_Receptacle_HRO_TYPE-C-31-M-12
- moved J1 1.49 mm to (13.1, 97.3)
Routing:
- net Net-(F1-Pad1): track 19.4 -> 23.4 mm
- net Net-(J1-CC2): track 2.09 -> 3.58 mm
- net Net-(J1-CC1): track 2.09 -> 3.58 mm
- net GNDU: vias 49 -> 51

Commit message: Rev B: build the top-scoring chaos lamp, and clear J1's silk from the edge
The lamp becomes candidate 1 of docs/lamp2: common anode at +3.75 V
(R16 15k), red fed from -y through 1.5k with x blended in through 8.2k
and +12 V through 8.2k, green from x through 24k, blue from z through
2.2k with -12 V through 36k.  Three resistors more than rev A, all
JLCPCB Basic parts; D1's footprint, place and angle are rev A's, which
its boards proved.  The symbol draws the dies blue, red, green so the
schematic's feeds still never cross.

check_circuit.py now reads the lamp back out of the netlist, checks it
is that wiring, and simulates it with the corrected LED model: 0.82 at
slow!, against rev A's 0.33.  Everything outside the lamp was compared
with rev A: all 204 other pins wire identically, the outline and
non-plated holes are byte-identical, and every routed net but the
lamp's and /SJ_Y (re-routed 1.2 mm lower near U1) is unchanged.

Also:
  * J1's silk stubs ended 0.15 mm from the edge, inside JLCPCB's 0.2 mm
    pull-back; trimmed to 0.45 mm.
  * The schematic checker now models KiCad reversing justification on
    rotated symbols' fields -- it had let six clashing labels through.
  * The eye filter is plain numpy again, so ./make.py needs only numpy
    and Pillow, as the README says.
  * The assembler notes gave D1's pin order as anticlockwise; it is
    clockwise.
  * Op-amp values hidden like the multipliers': "LF412 op-amp" says it.
  * Stock refreshed for the scarce parts; rev B, dated 2026-10-02.

Co-Authored-By: Claude Opus 5.5 <noreply@anthropic.com>
Claude-Session: https://claude.ai/code/session_01FyYQ1p4JtCVvJKRozbkYm7
Parts:
- added R22: 8.2k, Resistor_SMD:R_0805_2012Metric, F.Cu at (70.0, 60.5)
- added R23: 8.2k, Resistor_SMD:R_0805_2012Metric, F.Cu at (70.0, 63.5)
- added R24: 36k, Resistor_SMD:R_0805_2012Metric, F.Cu at (70.0, 53.5)
- R13: value 3.9k -> 24k
- R14: value 1.5k -> 2.2k
- R15: value 470R -> 1.5k
- R16: value 12k -> 15k
- TP6: value +3.2V -> +3.75V
- moved R14 4.50 mm to (70.0, 50.5), turned to 180 degrees
- moved R15 4.50 mm to (70.0, 57.5), turned to 180 degrees
- moved C18 2.24 mm to (63.0, 66.0)
- moved R13 1.50 mm to (70.0, 46.5), turned to 180 degrees
Connections:
- R14 pad 2: /-y -> /z
- R15 pad 2: /z -> /-y
Routing:
- net /x: track 190.5 -> 206.5 mm
- net -12V: track 174.7 -> 189.9 mm, vias 3 -> 4
- net /z: track 152.4 -> 140.0 mm, vias 7 -> 5
- net Net-(D1-A): track 33.9 -> 28.4 mm
- net Net-(D1-R): track 17.5 -> 20.4 mm
- net +12V: track 174.9 -> 176.9 mm
- net Net-(D1-B): track 13.0 -> 14.4 mm
- net Net-(D1-G): track 18.8 -> 17.6 mm
- net /-y: track 158.9 -> 159.9 mm
- net Net-(U2B-+): track 28.4 -> 29.4 mm
- net GND: vias 255 -> 248
Other:
- board text added: "-y (+x) = red"
- board text added: "2026-10-02 rev B"
- board text added: "PCB by Jason Gallicchio and Claude Opus 5 Max 2026-10-02 rev B"
- board text added: "z = blue"
- board text removed: "-y = blue"
- board text removed: "2026-09-15 rev A"
- board text removed: "PCB by Jason Gallicchio and Claude Opus 5 Max 2026-09-15 rev A"
- board text removed: "z = red"
